File: pcb/tone_trixter.kicad_sch (KiCad schematic)
At the start: 101 parts, among them J1 INA jack lead, J10 microSD DM3AT, J2 OUT jack lead, J3 DC 2.1mm lead, J4 Battery lead, J5 Enclosure bond, J6 OLED 1.3" 7-pin, J7 SW-L bypass, J8 INB jack lead, J9 SW-R tuner, SW1 PEC11R-4220F-S0024, U1 OPA1642AIDR, U2 OPA1642AIDR, U3 OPA1642AIDR, U4 Daisy Seed3

Commit message: pcb: fix Seed footprint (1x20 -> 2x20 Daisy) + deterministic UUIDs
U4 was assigned PinSocket_1x20 (20 pads) against a 40-pin Seed3 symbol,
so half the module was unconnected. Switch to Module:Electrosmith_Daisy_
Seed (40 pads, correct 2x20 geometry). Also make schematic UUIDs
deterministic (counter-based uuid5 in kisch.U) so regenerations stay
byte-identical and don't churn the PCB<->schematic link. ERC: 0 errors,
9 benign OPA library-copy warnings.

Co-Authored-By: Claude Opus 4.8 <noreply@anthropic.com>
Claude-Session: https://claude.ai/code/session_01GZEvjBMn4qYKgWYpBHDYwL
Parts:
- U4: footprint Connector_PinSocket_2.54mm:PinSocket_1x20_P2.54mm_Vertical -> Module:Electrosmith_Daisy_Seed

Commit message: pcb: first-pass K3599 board-mount jacks + placement script
- TT.pretty/K3599_TRS_6leg: first-pass footprint for the Mantech K3599
  (1/4in 3-cond closed/switched, 6 legs). Pads 1/2/3 = T/R/S (match the
  Conn_01x03 symbol), 3 unnumbered = switch legs (soldered, no net v1).
  ⚠ DIMS ARE GUESSES -- verify vs the real part before fab. fp-lib-table
  added for the TT footprint lib.
- gen_schematic: J1 (IN) and J2 (OUT) -> TT:K3599 (footprint swap only,
  no rewiring); J8 (internal Ch B) and J3 (DC) stay JST for now.
- gen_place.py: first-pass placement of the enclosure-constrained
  anchors (OLED, encoder, LEDs, jacks, footswitch/battery/bond
  connectors, Seed, SD) per the mock-up, with everything else staged in
  a grid to the right. Run with KiCad's python after a sync.
ERC: 0 errors, 9 benign OPA library-copy warnings.

Co-Authored-By: Claude Opus 4.8 <noreply@anthropic.com>
Claude-Session: https://claude.ai/code/session_01GZEvjBMn4qYKgWYpBHDYwL
Parts:
- J1: footprint Connector_JST:JST_XH_B3B-XH-A_1x03_P2.50mm_Vertical -> TT:K3599_TRS_6leg; Note IN jack, TRS switched, plastic body. pin1 tip · pin2 ring (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 -> IN jack, K3599 board-mount TRS switched, bottom-mounted. pi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
- J2: footprint Connector_JST:JST_XH_B3B-XH-A_1x03_P2.50mm_Vertical -> TT:K3599_TRS_6leg; Note OUT jack, TRS SWITCHED, plastic body: pin1 tip · pin2 ring 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 -> OUT jack, K3599 board-mount TRS switched, bottom-mounted: p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
Changed lines of the file:
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@@
     (property "Reference" "J1" (at 17.78 220.98000000000002 0) (effects (font (size 1.27 1.27))))
     (property "Value" "INA jack lead" (at 17.78 226.06 0) (effects (font (size 1.27 1.27))))
-    (property "Footprint" "Connector_JST:JST_XH_B3B-XH-A_1x03_P2.50mm_Vertical" (at 15.24 223.52 0) (effects (font (size 1.27 1.27)) (hide yes)))
+    (property "Footprint" "TT:K3599_TRS_6leg" (at 15.24 223.52 0) (effects (font (size 1.27 1.27)) (hide yes)))
     (property "Datasheet" "~" (at 15.24 223.52 0) (effects (font (size 1.27 1.27)) (hide yes)))
-    (property "Note" "IN jack, TRS switched, plastic body. pin1 tip · pin2 ring (sleeve–ring link AT THE JACK) · pin3 sleeve" (at 15.24 223.52 0) (effects (font (size 1.27 1.27)) (hide yes)))
+    (property "Note" "IN jack, K3599 board-mount TRS switched, bottom-mounted. pin1 tip · pin2 ring (sleeve–ring link AT THE JACK) · pin3 sleeve" (at 15.24 223.52 0) (effects (font (size 1.27 1.27)) (hide yes)))
     (pin "1")
     (pin "2")
@@
     (property "Reference" "J2" (at 220.98 347.97999999999996 0) (effects (font (size 1.27 1.27))))
     (property "Value" "OUT jack lead" (at 220.98 353.06 0) (effects (font (size 1.27 1.27))))
-    (property "Footprint" "Connector_JST:JST_XH_B3B-XH-A_1x03_P2.50mm_Vertical" (at 218.44 350.52 0) (effects (font (size 1.27 1.27)) (hide yes)))
+    (property "Footprint" "TT:K3599_TRS_6leg" (at 218.44 350.52 0) (effects (font (size 1.27 1.27)) (hide yes)))
     (property "Datasheet" "~" (at 218.44 350.52 0) (effects (font (size 1.27 1.27)) (hide yes)))
-    (property "Note" "OUT jack, TRS SWITCHED, plastic body: pin1 tip · pin2 ring = BATTERY − (switches the pedal on) · pin3 sleeve" (at 218.44 350.52 0) (effects (font (size 1.27 1.27)) (hide yes)))
-    (pin "1")
-    (pin "2")
+    (property "Note" "OUT jack, K3599 board-mount TRS switched, bottom-mounted: pin1 tip · pin2 ring = BATTERY − (switches the pedal on) · pin3 sleeve" (at 218.44 350.52 0) (effects (font (size 1.27 1.27)) (hide yes)))
+    (pin "1")
+    (pin "2")

Commit message: pcb: Channel B gets a real TRS jack (IN B), XLR reserve dropped
Reversed the v1 plan: instead of reserving a blind XLR cutout for a v2
mic, drill a second K3599 TRS (IN B) beside IN A now. J8 -> K3599
footprint on AIN2; the two instrument inputs are independent (IN A=AIN1,
IN B=AIN2), the AIN2 sharing is only IN B vs a future mic. J8 anchor
moved to the back wall next to IN A; mockup rear wall now IN B/IN A/DC/
USB/OUT (5 holes, no XLR). No analogue redesign -- U2 was already there.

Co-Authored-By: Claude Opus 4.8 <noreply@anthropic.com>
Parts:
- J8: footprint Connector_JST:JST_XH_B3B-XH-A_1x03_P2.50mm_Vertical -> TT:K3599_TRS_6leg; Note SECOND HIGH-Z CHANNEL — on the board only, NOT drilled in v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 -> IN B jack, K3599 board-mount TRS switched, bottom-mounted (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
Changed lines of the file:
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@@
     (property "Reference" "J8" (at 17.78 287.02 0) (effects (font (size 1.27 1.27))))
     (property "Value" "INB jack lead" (at 17.78 292.1 0) (effects (font (size 1.27 1.27))))
-    (property "Footprint" "Connector_JST:JST_XH_B3B-XH-A_1x03_P2.50mm_Vertical" (at 15.24 289.56 0) (effects (font (size 1.27 1.27)) (hide yes)))
+    (property "Footprint" "TT:K3599_TRS_6leg" (at 15.24 289.56 0) (effects (font (size 1.27 1.27)) (hide yes)))
     (property "Datasheet" "~" (at 15.24 289.56 0) (effects (font (size 1.27 1.27)) (hide yes)))
-    (property "Note" "SECOND HIGH-Z CHANNEL — on the board only, NOT drilled in v1 (brief §3.2)" (at 15.24 289.56 0) (effects (font (size 1.27 1.27)) (hide yes)))
+    (property "Note" "IN B jack, K3599 board-mount TRS switched, bottom-mounted (DRILLED in v1 — second high-Z instrument input, brief §3.2). pin1 tip · pin2 ring (sleeve–ring link AT THE JACK) · pin3 sleeve" (at 15.24 289.56 0) (effects (font (size 1.27 1.27)) (hide yes)))
     (pin "1")
     (pin "2")
