File: pcb/tone_trixter.kicad_sch (KiCad schematic)
At the start: 101 parts, among them J1 INA jack lead, J10 microSD DM3AT, J2 OUT jack lead, J3 DC 2.1mm lead, J4 Battery lead, J5 Enclosure bond, J6 OLED 1.3" 7-pin, J7 SW-L bypass, J8 INB jack lead, J9 SW-R tuner, SW1 PEC11R-4220F-S0024, U1 OPA1642AIDR, U2 OPA1642AIDR, U3 OPA1642AIDR, U4 Daisy Seed3

Commit message: pcb: restore point before left-right mirror fix
Snapshot of the current board + schematic before correcting a mirrored
placement. The 3D view (control side, player orientation) shows the
encoder/IN on the player's LEFT, but the validated paper panel template
has them on the RIGHT -- the board is a left-right mirror of the panel
(root cause: gen_place.py lacks the Y-flip gen_mockup_svg.py applies).

Includes the current hand placement, the VREF per-channel bypass caps
(C32/C33) and junction fix in gen_schematic.py. Committed as-is so the
mirror operation has a clean revert point.
Parts:
- added C32, C33: 100n, Capacitor_SMD:C_0805_2012Metric, symbol Device:C
Connections:
- net GNDA: now also C32.2, C33.2
- net VREF: now also C32.1, C33.1
Changed lines of the file:
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@@
   (junction (at 106.68 17.78) (diameter 0) (color 0 0 0 0))
   (junction (at 142.24 20.32) (diameter 0) (color 0 0 0 0))
+  (junction (at 25.4 220.98) (diameter 0) (color 0 0 0 0))
   (junction (at 41.91 220.98) (diameter 0) (color 0 0 0 0))
   (junction (at 60.96 220.98) (diameter 0) (color 0 0 0 0))
@@
   (junction (at 177.8 220.98) (diameter 0) (color 0 0 0 0))
   (junction (at 182.88 220.98) (diameter 0) (color 0 0 0 0))
+  (junction (at 25.4 287.02) (diameter 0) (color 0 0 0 0))
   (junction (at 41.91 287.02) (diameter 0) (color 0 0 0 0))
   (junction (at 60.96 287.02) (diameter 0) (color 0 0 0 0))
@@
   (wire (pts (xy 266.7 270.51) (xy 266.7 267.97)) (stroke (width 0) (type default)))
   (wire (pts (xy 314.96 287.02) (xy 317.5 287.02)) (stroke (width 0) (type default)))
+  (wire (pts (xy 49.53 241.3) (xy 49.53 238.76)) (stroke (width 0) (type default)))
+  (wire (pts (xy 49.53 307.34) (xy 49.53 304.8)) (stroke (width 0) (type default)))
   (text "POWER — parallel diode-OR (pinmap §4n), no regulator. VIN abs max 17 V: 12 V adapters yes, 18 V no." (exclude_from_sim no) (at 10.16 7.62 0) (effects (font (size 1.8 1.8)) (justify left bottom)))
   (text "Rail = VIN (≈8.6 V battery / ≈11.6 V adapter). Battery − returns via the OUT ring (the power switch)." (exclude_from_sim no) (at 10.16 50.8 0) (effects (font (size 1.4 1.4)) (justify left bottom)))
@@
   (global_label "SD_CD" (shape bidirectional) (at 261.62 284.48 180) (fields_autoplaced yes) (effects (font (size 1.27 1.27)) (justify right))
     (property "Intersheetrefs" "${INTERSHEET_REFS}" (at 261.62 284.48 0) (effects (font (size 1.27 1.27)) (hide yes)))
+  )
+  (global_label "VREF" (shape bidirectional) (at 49.53 238.76 90) (fields_autoplaced yes) (effects (font (size 1.27 1.27)) (justify left))
+    (property "Intersheetrefs" "${INTERSHEET_REFS}" (at 49.53 238.76 0) (effects (font (size 1.27 1.27)) (hide yes)))
+  )
+  (global_label "VREF" (shape bidirectional) (at 49.53 304.8 90) (fields_autoplaced yes) (effects (font (size 1.27 1.27)) (justify left))
+    (property "Intersheetrefs" "${INTERSHEET_REFS}" (at 49.53 304.8 0) (effects (font (size 1.27 1.27)) (hide yes)))
   )
   (symbol (lib_id "Connector:Conn_01x02_Pin") (at 15.24 20.32 0) (unit 1)
@@
     (pin "1")
     (instances (project "tone_trixter" (path "/03fac6e5-0644-5314-951c-6cda957413cd" (reference "#PWR") (unit 1))))
+  )
+  (symbol (lib_id "Device:C") (at 49.53 245.11 0) (unit 1)
+    (exclude_from_sim no) (in_bom yes) (on_board yes) (dnp no)
+    (property "Reference" "C32" (at 52.07 242.57000000000002 0) (effects (font (size 1.27 1.27))))
+    (property "Value" "100n" (at 52.07 247.65 0) (effects (font (size 1.27 1.27))))
+    (property "Footprint" "Capacitor_SMD:C_0805_2012Metric" (at 49.53 245.11 0) (effects (font (size 1.27 1.27)) (hide yes)))
+    (property "Datasheet" "~" (at 49.53 245.11 0) (effects (font (size 1.27 1.27)) (hide yes)))
+    (property "Note" "ch A local VREF bypass — place beside the 1M VREF tap at the input (added 2026-10-21)" (at 49.53 245.11 0) (effects (font (size 1.27 1.27)) (hide yes)))
+    (pin "1")
+    (pin "2")
+    (instances (project "tone_trixter" (path "/03fac6e5-0644-5314-951c-6cda957413cd" (reference "C32") (unit 1))))
+  )
+  (symbol (lib_id "power:GNDA") (at 49.53 248.92 0) (unit 1)
+    (exclude_from_sim no) (in_bom no) (on_board yes) (dnp no)
+    (property "Reference" "#PWR" (at 52.07 246.38 0) (effects (font (size 1.27 1.27)) (hide yes)))
+    (property "Value" "GNDA" (at 52.07 251.45999999999998 0) (effects (font (size 1.27 1.27)) (hide yes)))
+    (property "Footprint" "" (at 49.53 248.92 0) (effects (font (size 1.27 1.27)) (hide yes)))
+    (property "Datasheet" "~" (at 49.53 248.92 0) (effects (font (size 1.27 1.27)) (hide yes)))
+    (pin "1")
+    (instances (project "tone_trixter" (path "/03fac6e5-0644-5314-951c-6cda957413cd" (reference "#PWR") (unit 1))))
+  )
+  (symbol (lib_id "Device:C") (at 49.53 311.15 0) (unit 1)
+    (exclude_from_sim no) (in_bom yes) (on_board yes) (dnp no)
+    (property "Reference" "C33" (at 52.07 308.60999999999996 0) (effects (font (size 1.27 1.27))))
+    (property "Value" "100n" (at 52.07 313.69 0) (effects (font (size 1.27 1.27))))
+    (property "Footprint" "Capacitor_SMD:C_0805_2012Metric" (at 49.53 311.15 0) (effects (font (size 1.27 1.27)) (hide yes)))
+    (property "Datasheet" "~" (at 49.53 311.15 0) (effects (font (size 1.27 1.27)) (hide yes)))
+    (property "Note" "ch B local VREF bypass — place beside the 1M VREF tap at the input (added 2026-10-21)" (at 49.53 311.15 0) (effects (font (size 1.27 1.27)) (hide yes)))
+    (pin "1")
+    (pin "2")
+    (instances (project "tone_trixter" (path "/03fac6e5-0644-5314-951c-6cda957413cd" (reference "C33") (unit 1))))
+  )
+  (symbol (lib_id "power:GNDA") (at 49.53 314.96 0) (unit 1)
+    (exclude_from_sim no) (in_bom no) (on_board yes) (dnp no)
+    (property "Reference" "#PWR" (at 52.07 312.41999999999996 0) (effects (font (size 1.27 1.27)) (hide yes)))
+    (property "Value" "GNDA" (at 52.07 317.5 0) (effects (font (size 1.27 1.27)) (hide yes)))
+    (property "Footprint" "" (at 49.53 314.96 0) (effects (font (size 1.27 1.27)) (hide yes)))
+    (property "Datasheet" "~" (at 49.53 314.96 0) (effects (font (size 1.27 1.27)) (hide yes)))
+    (pin "1")
+    (instances (project "tone_trixter" (path "/03fac6e5-0644-5314-951c-6cda957413cd" (reference "#PWR") (unit 1))))
