File: pcb/tone_trixter.kicad_sch (KiCad schematic)
At the start: 103 parts, among them J1 INA jack lead, J10 microSD DM3AT, J2 OUT jack lead, J3 DC 2.1mm lead, J4 Battery lead, J5 Enclosure bond, J6 OLED 1.3" 7-pin, J7 SW-L bypass, J8 INB jack lead, J9 SW-R tuner, SW1 PEC11R-4220F-S0024, U1 OPA1642AIDR, U2 OPA1642AIDR, U3 OPA1642AIDR, U4 Daisy Seed3

Commit message: pcb: output coupling caps to 1u C0G, LED/power/star placement pass
- gen_schematic: output C19/C21 10u film -> 1u C0G 1210 so they tuck
  under the OUT jack (C21->J2 tip run 3.0mm), matching the input caps
- LEDs D4/D5 forward to y=33.5 to clear the Daisy 2x20 pin field;
  silk alignment marks moved with them
- GND star (NT1) to the analog side, 6mm from the Daisy GNDA pin
- CH-B relaid under IN B (tip run 3.2mm); power section moved clear of
  the high-Z inputs (>=38mm) and out of the Daisy->USB corridor
- mirror_board_x.py: one-time X-mirror that set board handedness

Co-Authored-By: Claude Opus 4.8 <noreply@anthropic.com>
Parts:
- C11, C5: value 10u film -> 330n; footprint Capacitor_THT:C_Rect_L7.2mm_W7.2mm_P5.00mm_FKS2_FKP2_MKS2_MKP2 -> Capacitor_SMD:C_0805_2012Metric; Note (none) -> C0G/NP0 0805 (was 10u film); LF corner is set by the piezo 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
- C14, C8: value 10u film -> 1u; footprint Capacitor_THT:C_Rect_L7.2mm_W7.2mm_P5.00mm_FKS2_FKP2_MKS2_MKP2 -> Capacitor_SMD:C_1210_3225Metric; Note (none) -> C0G/NP0 1210 (was 10u film); inter-stage coupling into the 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
- C19: value 10u film -> 1u; footprint Capacitor_THT:C_Rect_L7.2mm_W7.2mm_P5.00mm_FKS2_FKP2_MKS2_MKP2 -> Capacitor_SMD:C_1210_3225Metric; Note (none) -> C0G/NP0 1210 (was 10u film); output-stage input coupling, A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
- C21: value 10u film -> 1u; footprint Capacitor_THT:C_Rect_L7.2mm_W7.2mm_P5.00mm_FKS2_FKP2_MKS2_MKP2 -> Capacitor_SMD:C_1210_3225Metric; Note (none) -> C0G/NP0 1210 (was 10u film); output coupling to the OUT jac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
Changed lines of the file:
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@@
     (exclude_from_sim no) (in_bom yes) (on_board yes) (dnp no)
     (property "Reference" "C5" (at 35.56 218.44 0) (effects (font (size 1.27 1.27))))
-    (property "Value" "10u film" (at 35.56 223.51999999999998 0) (effects (font (size 1.27 1.27))))
-    (property "Footprint" "Capacitor_THT:C_Rect_L7.2mm_W7.2mm_P5.00mm_FKS2_FKP2_MKS2_MKP2" (at 33.02 220.98 0) (effects (font (size 1.27 1.27)) (hide yes)))
+    (property "Value" "330n" (at 35.56 223.51999999999998 0) (effects (font (size 1.27 1.27))))
+    (property "Footprint" "Capacitor_SMD:C_0805_2012Metric" (at 33.02 220.98 0) (effects (font (size 1.27 1.27)) (hide yes)))
     (property "Datasheet" "~" (at 33.02 220.98 0) (effects (font (size 1.27 1.27)) (hide yes)))
+    (property "Note" "C0G/NP0 0805 (was 10u film); LF corner is set by the piezo 24.5n into 1M, so this value is ~irrelevant down to ~100n; small/low-profile fits under the TRS jack" (at 33.02 220.98 0) (effects (font (size 1.27 1.27)) (hide yes)))
     (pin "1")
     (pin "2")
@@
     (exclude_from_sim no) (in_bom yes) (on_board yes) (dnp no)
     (property "Reference" "C8" (at 123.19000000000001 220.98000000000002 0) (effects (font (size 1.27 1.27))))
-    (property "Value" "10u film" (at 123.19000000000001 226.06 0) (effects (font (size 1.27 1.27))))
-    (property "Footprint" "Capacitor_THT:C_Rect_L7.2mm_W7.2mm_P5.00mm_FKS2_FKP2_MKS2_MKP2" (at 120.65 223.52 0) (effects (font (size 1.27 1.27)) (hide yes)))
+    (property "Value" "1u" (at 123.19000000000001 226.06 0) (effects (font (size 1.27 1.27))))
+    (property "Footprint" "Capacitor_SMD:C_1210_3225Metric" (at 120.65 223.52 0) (effects (font (size 1.27 1.27)) (hide yes)))
     (property "Datasheet" "~" (at 120.65 223.52 0) (effects (font (size 1.27 1.27)) (hide yes)))
+    (property "Note" "C0G/NP0 1210 (was 10u film); inter-stage coupling into the 10k inverting input, corner 1/(2pi*10k*1u)=16Hz -- keep >=1u" (at 120.65 223.52 0) (effects (font (size 1.27 1.27)) (hide yes)))
     (pin "1")
     (pin "2")
@@
     (exclude_from_sim no) (in_bom yes) (on_board yes) (dnp no)
     (property "Reference" "C11" (at 35.56 284.47999999999996 0) (effects (font (size 1.27 1.27))))
-    (property "Value" "10u film" (at 35.56 289.56 0) (effects (font (size 1.27 1.27))))
-    (property "Footprint" "Capacitor_THT:C_Rect_L7.2mm_W7.2mm_P5.00mm_FKS2_FKP2_MKS2_MKP2" (at 33.02 287.02 0) (effects (font (size 1.27 1.27)) (hide yes)))
+    (property "Value" "330n" (at 35.56 289.56 0) (effects (font (size 1.27 1.27))))
+    (property "Footprint" "Capacitor_SMD:C_0805_2012Metric" (at 33.02 287.02 0) (effects (font (size 1.27 1.27)) (hide yes)))
     (property "Datasheet" "~" (at 33.02 287.02 0) (effects (font (size 1.27 1.27)) (hide yes)))
+    (property "Note" "C0G/NP0 0805 (was 10u film); LF corner is set by the piezo 24.5n into 1M, so this value is ~irrelevant down to ~100n; small/low-profile fits under the TRS jack" (at 33.02 287.02 0) (effects (font (size 1.27 1.27)) (hide yes)))
     (pin "1")
     (pin "2")
@@
     (exclude_from_sim no) (in_bom yes) (on_board yes) (dnp no)
     (property "Reference" "C14" (at 123.19000000000001 287.02 0) (effects (font (size 1.27 1.27))))
-    (property "Value" "10u film" (at 123.19000000000001 292.1 0) (effects (font (size 1.27 1.27))))
-    (property "Footprint" "Capacitor_THT:C_Rect_L7.2mm_W7.2mm_P5.00mm_FKS2_FKP2_MKS2_MKP2" (at 120.65 289.56 0) (effects (font (size 1.27 1.27)) (hide yes)))
+    (property "Value" "1u" (at 123.19000000000001 292.1 0) (effects (font (size 1.27 1.27))))
+    (property "Footprint" "Capacitor_SMD:C_1210_3225Metric" (at 120.65 289.56 0) (effects (font (size 1.27 1.27)) (hide yes)))
     (property "Datasheet" "~" (at 120.65 289.56 0) (effects (font (size 1.27 1.27)) (hide yes)))
+    (property "Note" "C0G/NP0 1210 (was 10u film); inter-stage coupling into the 10k inverting input, corner 1/(2pi*10k*1u)=16Hz -- keep >=1u" (at 120.65 289.56 0) (effects (font (size 1.27 1.27)) (hide yes)))
     (pin "1")
     (pin "2")
@@
     (exclude_from_sim no) (in_bom yes) (on_board yes) (dnp no)
     (property "Reference" "C19" (at 127.0 353.06 0) (effects (font (size 1.27 1.27))))
-    (property "Value" "10u film" (at 127.0 358.14000000000004 0) (effects (font (size 1.27 1.27))))
-    (property "Footprint" "Capacitor_THT:C_Rect_L7.2mm_W7.2mm_P5.00mm_FKS2_FKP2_MKS2_MKP2" (at 124.46 355.6 0) (effects (font (size 1.27 1.27)) (hide yes)))
+    (property "Value" "1u" (at 127.0 358.14000000000004 0) (effects (font (size 1.27 1.27))))
+    (property "Footprint" "Capacitor_SMD:C_1210_3225Metric" (at 124.46 355.6 0) (effects (font (size 1.27 1.27)) (hide yes)))
     (property "Datasheet" "~" (at 124.46 355.6 0) (effects (font (size 1.27 1.27)) (hide yes)))
+    (property "Note" "C0G/NP0 1210 (was 10u film); output-stage input coupling, AOUT1 into 15k -> corner 1/(2pi*15k*1u)=10.6Hz; small/low-profile fits under the OUT jack" (at 124.46 355.6 0) (effects (font (size 1.27 1.27)) (hide yes)))
     (pin "1")
     (pin "2")
@@
     (exclude_from_sim no) (in_bom yes) (on_board yes) (dnp no)
     (property "Reference" "C21" (at 189.23 350.52 0) (effects (font (size 1.27 1.27))))
-    (property "Value" "10u film" (at 189.23 355.6 0) (effects (font (size 1.27 1.27))))
-    (property "Footprint" "Capacitor_THT:C_Rect_L7.2mm_W7.2mm_P5.00mm_FKS2_FKP2_MKS2_MKP2" (at 186.69 353.06 0) (effects (font (size 1.27 1.27)) (hide yes)))
+    (property "Value" "1u" (at 189.23 355.6 0) (effects (font (size 1.27 1.27))))
+    (property "Footprint" "Capacitor_SMD:C_1210_3225Metric" (at 186.69 353.06 0) (effects (font (size 1.27 1.27)) (hide yes)))
     (property "Datasheet" "~" (at 186.69 353.06 0) (effects (font (size 1.27 1.27)) (hide yes)))
-    (pin "1")
-    (pin "2")
+    (property "Note" "C0G/NP0 1210 (was 10u film); output coupling to the OUT jack, drives amp input (>=470k) -> corner <1Hz; small/low-profile fits under J2" (at 186.69 353.06 0) (effects (font (size 1.27 1.27)) (hide yes)))
+    (pin "1")
+    (pin "2")
